File: PCB/FancyPantsMkII.sch (KiCad schematic (older format))
At the start: 11 parts, among them IC1 ATMEGA1284P-P, J1 J_SIGNAL, J2 J_DISPLAY, Y1 16MHz

Commit message: fixed display reset net name
display reset net was named same as uC reset net, tying the two
together. Will probably never remake this board, but needed to fix the
net in case anyone else ever wants to.
Connections:
- net labels added: DISP_RST
Changed lines of the file:
@@
 LIBS:w_device
 LIBS:ML_Kicad
+LIBS:FancyPantsMkII-cache
 EELAYER 27 0
 EELAYER END
@@
 Sheet 1 1
 Title ""
-Date "30 dec 2013"
+Date "18 feb 2014"
 Rev ""
 Comp ""
@@
 SCL
 Text GLabel 6050 3600 0    30   Input ~ 0
-RST
+DISP_RST
 Text GLabel 3100 4700 2    30   Input ~ 0
-RST
+DISP_RST
 Wire Wire Line
 	3050 4700 3100 4700
